Commit message: gripper coloured and add missing joint to make it work

File: ezgripper_driver/urdf/ezgripper_dual_gen2_articulated.urdf.xacro (robot description, xacro)
@@ -22,4 +22,7 @@
     </inertial>
     </link>
+    <gazebo reference="${prefix}_ezgripper_palm_link">
+      <material>Gazebo/BlueLaser</material>
+    </gazebo>
     <joint name="${prefix}_ezgripper_connect" type="fixed">
         <xacro:insert_block name="origin" />
@@ -40,4 +43,10 @@
     <ezgripper_knuckle_trans prefix="${prefix}" postfix="L1_L2_1"/>
     <gazebo_knuckle_jsp prefix="${prefix}" />
+    <joint name="${prefix}_ezgripper_ee_fixed_joint" type="fixed">
+      <parent link="${prefix}_ezgripper_palm_link" />
+      <child link = "eg_manipulator" />
+      <origin xyz="0.0 0.0 0.10" rpy="0.0 0.0 0.0" />
+    </joint>
+    <link name="eg_manipulator" />
 </xacro:macro>
 <xacro:macro name="ezgripper_finger_L1" params="prefix postfix reflect">
@@ -60,4 +69,7 @@
       </inertial>
     </link>
+    <gazebo reference="${prefix}_ezgripper_finger_L1_${postfix}">
+      <material>Gazebo/White</material>
+    </gazebo>
 </xacro:macro>
 <xacro:macro name="ezgripper_finger_L2" params="prefix postfix reflect">
@@ -80,4 +92,7 @@
       </inertial>
     </link>
+    <gazebo reference="${prefix}_ezgripper_finger_L2_${postfix}">
+      <material>Gazebo/White</material>
+    </gazebo>
 </xacro:macro>
     <!-- joints -->
@@ -123,5 +138,5 @@
    <gazebo>
      <plugin name="joint_state_publisher" filename="libgazebo_ros_joint_state_publisher.so">
-       <jointName>${prefix}_ezgripper_knuckle_L1_L2_1,${prefix}_ezgripper_knuckle_L1_L2_2</jointName>
+       <jointName>${prefix}_ezgripper_knuckle_L1_L2_1,${prefix}_ezgripper_knuckle_L1_L2_2, ${prefix}_ezgripper_knuckle_palm_L1_1 </jointName>
      </plugin>
    </gazebo>

Commit message: add color for RVIZ

File: ezgripper_driver/urdf/ezgripper_dual_gen2_articulated.urdf.xacro (robot description, xacro)
@@ -2,4 +2,10 @@
 <robot name="ezgripper" xmlns:xacro="http://ros.org/wiki/xacro">
 <!--xacro:macro name="ezgripper" params="*origin"-->
+<material name="blue">
+    <color rgba = "0.19 0.22 0.99 1.0"/>
+</material>
+<material name="white">
+    <color rgba = "1.0 1.0 1.0 1.0"/>
+</material>
 <xacro:macro name="ezgripper_dual" params="prefix parent_link *origin">
     <!-- links -->
@@ -10,4 +16,5 @@
           <mesh filename="package://ezgripper_driver/meshes/ezgripper_gen2/SAKE_Palm_Dual_Gen2.stl"/>
         </geometry>
+        <material name="blue"/>
       </visual>
       <collision>
@@ -46,5 +53,5 @@
       <parent link="${prefix}_ezgripper_palm_link" />
       <child link = "eg_manipulator" />
-      <origin xyz="0.0 0.0 0.10" rpy="0.0 0.0 0.0" />
+      <origin xyz="0.083 0.0 0.0" rpy="1.570796325 3.14159265 1.570796325" />
     </joint>
     <link name="eg_manipulator" />
@@ -57,4 +64,5 @@
           <mesh filename="package://ezgripper_driver/meshes/ezgripper_gen2/SAKE_Finger_L1_Gen2.stl"/>
         </geometry>
+        <material name="white"/>
       </visual>
       <collision>
@@ -63,4 +71,5 @@
           <mesh filename="package://ezgripper_driver/meshes/ezgripper_gen2/SAKE_Finger_L1_Gen2.stl"/>
         </geometry>
+        <material name="white"/>
       </collision>
       <inertial>
@@ -80,4 +89,5 @@
           <mesh filename="package://ezgripper_driver/meshes/ezgripper_gen2/SAKE_Finger_L2_Gen2.stl"/>
         </geometry>
+        <material name="white"/>
       </visual>
       <collision>
@@ -86,4 +96,5 @@
           <mesh filename="package://ezgripper_driver/meshes/ezgripper_gen2/SAKE_Finger_L2_Gen2.stl"/>
         </geometry>
+        <material name="white"/>
       </collision>
       <inertial>

Commit message: working xacro file allowing moveit and gazebo control

File: ezgripper_driver/urdf/ezgripper_dual_gen2_articulated.urdf.xacro (robot description, xacro)
@@ -34,5 +34,4 @@
     <joint name="${prefix}_ezgripper_connect" type="fixed">
         <xacro:insert_block name="origin" />
-        <!-- <origin rpy="0 0 0" xyz="0.049 0.0 0.2"/> -->
         <parent link="${parent_link}"/>
         <child link="${prefix}_ezgripper_palm_link"/>
@@ -48,5 +47,6 @@
     <ezgripper_knuckle_L1_L2 prefix="${prefix}" postfix="1" reflectY="1" reflectZ="1" reflectR="-1" mimic_test="false"/>
     <ezgripper_knuckle_L1_L2 prefix="${prefix}" postfix="2" reflectY="-1" reflectZ="1" reflectR="1" mimic_test="true"/>
-    <ezgripper_knuckle_trans prefix="${prefix}" postfix="L1_L2_1"/>
+    <ezgripper_knuckle_trans prefix="${prefix}" postfix="1"/>
+    <ezgripper_knuckle_trans prefix="${prefix}" postfix="2"/>
     <gazebo_knuckle_jsp prefix="${prefix}" />
     <joint name="${prefix}_ezgripper_ee_fixed_joint" type="fixed">
@@ -107,5 +107,5 @@
     </gazebo>
 </xacro:macro>
-    <!-- joints -->
+<!-- joints -->
 <xacro:macro name="ezgripper_knuckle_palm_L1" params="prefix postfix reflectY reflectZ reflectR mimic_test">
     <joint name="${prefix}_ezgripper_knuckle_palm_L1_${postfix}" type="revolute">
@@ -115,7 +115,4 @@
       <axis xyz="0 1 0"/>
       <limit lower="0" upper="1.94" effort="1" velocity="3.67"/>
-      <xacro:if value="${mimic_test}">
-           <mimic joint="${prefix}_ezgripper_knuckle_palm_L1_1"/>
-      </xacro:if>
     </joint>
 </xacro:macro>
@@ -125,5 +122,4 @@
       <child link="${prefix}_ezgripper_finger_L2_${postfix}"/>
       <origin xyz="0.052 0 0" rpy="0 0 0"/>
-      <!-- origin xyz="0.06 0 0" rpy="${3.14159 * reflectR} 0 0"/-->
       <axis xyz="0 1 0"/>
       <limit lower="0" upper="1.94" effort="1" velocity="3.67"/>
@@ -137,5 +133,5 @@
    <transmission name="${prefix}_ezgripper_trans_${postfix}">
       <type>transmission_interface/SimpleTransmission</type>
-      <joint name="${prefix}_ezgripper_knuckle_${postfix}">
+      <joint name="${prefix}_ezgripper_knuckle_palm_L1_${postfix}">
          <hardwareInterface>hardware_interface/PositionJointInterface</hardwareInterface>
       </joint>
@@ -149,11 +145,12 @@
    <gazebo>
      <plugin name="joint_state_publisher" filename="libgazebo_ros_joint_state_publisher.so">
-       <jointName>${prefix}_ezgripper_knuckle_L1_L2_1,${prefix}_ezgripper_knuckle_L1_L2_2, ${prefix}_ezgripper_knuckle_palm_L1_1 </jointName>
+       <jointName>${prefix}_ezgripper_knuckle_L1_L2_1,${prefix}_ezgripper_knuckle_L1_L2_2, ${prefix}_ezgripper_knuckle_palm_L1_1, ${prefix}_ezgripper_knuckle_palm_L1_2 </jointName>
      </plugin>
    </gazebo>
 </xacro:macro>
 <gazebo>
-   <plugin name="gazebo_ros_control" filename="libgazebo_ros_control.so">
-   </plugin>
+ <plugin name="ros_control" filename="libgazebo_ros_control.so">
+   <robotSimType>gazebo_ros_control/DefaultRobotHWSim</robotSimType>
+ </plugin>
 </gazebo>
 </robot>

Commit message: fix the revolute part

File: ezgripper_driver/urdf/ezgripper_dual_gen2_articulated.urdf.xacro (robot description, xacro)
@@ -118,5 +118,5 @@
 </xacro:macro>
 <xacro:macro name="ezgripper_knuckle_L1_L2" params="prefix postfix reflectY reflectZ reflectR mimic_test">
-    <joint name="${prefix}_ezgripper_knuckle_L1_L2_${postfix}" type="revolute">
+    <joint name="${prefix}_ezgripper_knuckle_L1_L2_${postfix}" type="fixed">
       <parent link="${prefix}_ezgripper_finger_L1_${postfix}"/>
       <child link="${prefix}_ezgripper_finger_L2_${postfix}"/>
@@ -145,5 +145,5 @@
    <gazebo>
      <plugin name="joint_state_publisher" filename="libgazebo_ros_joint_state_publisher.so">
-       <jointName>${prefix}_ezgripper_knuckle_L1_L2_1,${prefix}_ezgripper_knuckle_L1_L2_2, ${prefix}_ezgripper_knuckle_palm_L1_1, ${prefix}_ezgripper_knuckle_palm_L1_2 </jointName>
+       <jointName>${prefix}_ezgripper_knuckle_palm_L1_1, ${prefix}_ezgripper_knuckle_palm_L1_2 </jointName>
      </plugin>
    </gazebo>

Commit message: make urdf compatible with gazebo and mimic joints

File: ezgripper_driver/urdf/ezgripper_dual_gen2_articulated.urdf.xacro (robot description, xacro)
@@ -1,5 +1,4 @@
 <?xml version="1.0" encoding="UTF-8"?>
 <robot name="ezgripper" xmlns:xacro="http://ros.org/wiki/xacro">
-<!--xacro:macro name="ezgripper" params="*origin"-->
 <material name="blue">
     <color rgba = "0.19 0.22 0.99 1.0"/>
@@ -45,8 +44,8 @@
     <ezgripper_knuckle_palm_L1 prefix="${prefix}" postfix="1" reflectY="1" reflectZ="1" reflectR="1" mimic_test="false"/>
     <ezgripper_knuckle_palm_L1 prefix="${prefix}" postfix="2" reflectY="-1" reflectZ="1" reflectR="-1" mimic_test="true"/>
+    <mimic_joint_plugin_gazebo prefix="${prefix}"/>
     <ezgripper_knuckle_L1_L2 prefix="${prefix}" postfix="1" reflectY="1" reflectZ="1" reflectR="-1" mimic_test="false"/>
     <ezgripper_knuckle_L1_L2 prefix="${prefix}" postfix="2" reflectY="-1" reflectZ="1" reflectR="1" mimic_test="true"/>
-    <ezgripper_knuckle_trans prefix="${prefix}" postfix="1"/>
-    <ezgripper_knuckle_trans prefix="${prefix}" postfix="2"/>
+    <ezgripper_knuckle_trans prefix="${prefix}" postfix="palm_L1_1"/>
     <gazebo_knuckle_jsp prefix="${prefix}" />
     <joint name="${prefix}_ezgripper_ee_fixed_joint" type="fixed">
@@ -115,4 +114,7 @@
       <axis xyz="0 1 0"/>
       <limit lower="0" upper="1.94" effort="1" velocity="3.67"/>
+      <xacro:if value="${mimic_test}">
+          <mimic joint="${prefix}_ezgripper_knuckle_palm_L1_1" multiplier="1.0" offset="0.0"/>
+      </xacro:if>
     </joint>
 </xacro:macro>
@@ -125,27 +127,39 @@
       <limit lower="0" upper="1.94" effort="1" velocity="3.67"/>
       <xacro:if value="${mimic_test}">
-           <mimic joint="${prefix}_ezgripper_knuckle_L1_L2_1"/>
+           <mimic joint="${prefix}_ezgripper_knuckle_L1_L2_1" multiplier="1.0" offset="0.0"/>
       </xacro:if>
     </joint>
 </xacro:macro>
     <!-- transmissions for Gazebo -->
-<xacro:macro name="ezgripper_knuckle_trans" params="prefix postfix">
-   <transmission name="${prefix}_ezgripper_trans_${postfix}">
-      <type>transmission_interface/SimpleTransmission</type>
-      <joint name="${prefix}_ezgripper_knuckle_palm_L1_${postfix}">
-         <hardwareInterface>hardware_interface/PositionJointInterface</hardwareInterface>
-      </joint>
-      <actuator name="${prefix}_ezgripper_motor${postfix}">
-         <mechanicalReduction>1</mechanicalReduction>
-         <hardwareInterface>hardware_interface/PositionJointInterface</hardwareInterface>
-      </actuator>
-   </transmission>
-</xacro:macro>
-<xacro:macro name="gazebo_knuckle_jsp" params="prefix">
-   <gazebo>
-     <plugin name="joint_state_publisher" filename="libgazebo_ros_joint_state_publisher.so">
-       <jointName>${prefix}_ezgripper_knuckle_palm_L1_1, ${prefix}_ezgripper_knuckle_palm_L1_2 </jointName>
-     </plugin>
-   </gazebo>
+    <xacro:macro name="ezgripper_knuckle_trans" params="prefix postfix">
+       <transmission name="${prefix}_ezgripper_trans_${postfix}">
+          <type>transmission_interface/SimpleTransmission</type>
+          <joint name="${prefix}_ezgripper_knuckle_${postfix}">
+             <hardwareInterface>hardware_interface/PositionJointInterface</hardwareInterface>
+          </joint>
+          <actuator name="${prefix}_ezgripper_motor${postfix}">
+             <mechanicalReduction>1</mechanicalReduction>
+             <hardwareInterface>hardware_interface/PositionJointInterface</hardwareInterface>
+          </actuator>
+       </transmission>
+    </xacro:macro>
+    <xacro:macro name="gazebo_knuckle_jsp" params="prefix">
+       <gazebo>
+         <plugin name="joint_state_publisher" filename="libgazebo_ros_joint_state_publisher.so">
+           <jointName>${prefix}_ezgripper_knuckle_palm_L1_1</jointName>
+         </plugin>
+       </gazebo>
+    </xacro:macro>
+<xacro:macro name="mimic_joint_plugin_gazebo" params="prefix">
+  <gazebo>
+    <plugin name="mimic_joint_plugin" filename="libroboticsgroup_gazebo_mimic_joint_plugin.so">
+      <joint>${prefix}_ezgripper_knuckle_palm_L1_1</joint>
+      <mimicJoint>${prefix}_ezgripper_knuckle_palm_L1_2</mimicJoint>
+      <multiplier>1.0</multiplier>
+      <offset>0</offset>
+      <sensitiveness>0.0</sensitiveness>   <!-- if absolute difference between setpoint and process value is below this threshold, do nothing; 0.0 = disable [rad] -->
+      <maxEffort>1.0</maxEffort>
+    </plugin>
+  </gazebo>
 </xacro:macro>
 <gazebo>
